Commit message: update the shelf to add the side

File: urdf/shelf.urdf.xacro (robot description, xacro)
@@ -26,20 +26,13 @@
   </joint>
   <link name="base_link">
-<!--
-    <inertial>
-      <origin rpy="${M_PI/2} 0 0" xyz="0 0 0"/>
-      <mass value="1.0"/>
-      <inertia ixx="0.051828" ixy="0.0" ixz="0.0" iyy="0.088812" iyz="0.00012" izz="0.04517"/>
-    </inertial>
--->
     <inertial>
       <origin rpy="${M_PI/2} 0 0" xyz="0 0 0"/>
       <mass value="200.0"/>
-      <inertia ixx="0.0052406" ixy="0.0" ixz="0.0" iyy="0.0095404" iyz="0.00000025838" izz="0.004385"/>
+      <inertia ixx="0.051828" ixy="0.0" ixz="0.0" iyy="0.1050" iyz="0.0" izz="0.045472"/>
     </inertial>
     <visual>
       <origin xyz="0 0 0" rpy="${M_PI/2} 0 0" />
         <geometry>
-          <mesh filename="package://agv2_description/meshes/pallet_spring_supp_brk_100kg_with_top.stl" scale="0.001 0.001 0.001"/>
+          <mesh filename="package://agv2_description/meshes/pallet_spring_supp_brk_100kg_with_top_side.stl" scale="0.001 0.001 0.001"/>
         </geometry>
     </visual>
@@ -47,5 +40,5 @@
       <origin xyz="0 0 0" rpy="${M_PI/2} 0 0" />
         <geometry>
-          <mesh filename="package://agv2_description/meshes/pallet_spring_supp_brk_100kg_with_top.stl" scale="0.001 0.001 0.001"/>
+          <mesh filename="package://agv2_description/meshes/pallet_spring_supp_brk_100kg_with_top_side.stl" scale="0.001 0.001 0.001"/>
         </geometry>
     </collision>
