Commit message: move dummy loclation into the xacro

File: urdf/agv2.urdf.xacro (robot description, xacro)
@@ -54,15 +54,11 @@
     <origin rpy="-6.123E-17 0 0" xyz="${BASE_R*-1} 0.0 ${drive_wheel_r - agv_height/2 - hollow_h}" />
   </xacro:wheel>
-  <xacro:dummy_wheel name="lf_wheel" parent="base_link">
-    <origin rpy="-6.123E-17 0 0" xyz="${BASE_DUMMY_R} ${0.4275 + shaft_w/2 - 0.01} ${shaft_h/2 + dummy_r - agv_height/2 - hollow_h}" />
+  <xacro:dummy_wheel name="lf_wheel" parent="base_link" x_loc="${BASE_DUMMY_R}" y_loc="0.4275">
   </xacro:dummy_wheel>
-  <xacro:dummy_wheel name="rf_wheel" parent="base_link">
-    <origin rpy="-6.123E-17 0 0" xyz="${BASE_DUMMY_R*-1} ${0.4275 + shaft_w/2 - 0.01}  ${shaft_h/2 + dummy_r - agv_height/2 - hollow_h}" />
+  <xacro:dummy_wheel name="rf_wheel" parent="base_link" x_loc="${BASE_DUMMY_R*-1}" y_loc="0.4275">
   </xacro:dummy_wheel>
-  <xacro:dummy_wheel name="lr_wheel" parent="base_link">
-    <origin rpy="-6.123E-17 0 0" xyz="${BASE_DUMMY_R} ${-0.42475 + shaft_w/2 - 0.01}  ${shaft_h/2 + dummy_r - agv_height/2 - hollow_h}" />
+  <xacro:dummy_wheel name="lr_wheel" parent="base_link" x_loc="${BASE_DUMMY_R}" y_loc="-0.42475">
   </xacro:dummy_wheel>
-  <xacro:dummy_wheel name="rr_wheel" parent="base_link">
-    <origin rpy="-6.123E-17 0 0" xyz="${BASE_DUMMY_R*-1} ${-0.42475 + shaft_w/2 - 0.01} ${shaft_h/2 + dummy_r - agv_height/2 - hollow_h}" />
+  <xacro:dummy_wheel name="rr_wheel" parent="base_link" x_loc="${BASE_DUMMY_R*-1}" y_loc="-0.42475">
   </xacro:dummy_wheel>
 <!--

File: urdf/wheel_agv.urdf.xacro (robot description, xacro)
@@ -33,5 +33,5 @@
   <property name="shaft_h" value="0.0695" />
   <property name="shaft_w" value="0.033" />
-  <xacro:macro name="dummy_wheel" params="name parent *origin">
+  <xacro:macro name="dummy_wheel" params="name parent x_loc y_loc">
     <link name="${name}_shaft_link">
         <xacro:box_inertial mass="0.1" x="${shaft_w}" y="${dummy_w}" z="${shaft_h}">
@@ -78,5 +78,5 @@
     </link>
     <joint name="${name}_joint_shaft" type="continuous">
-      <insert_block name="origin" />
+      <origin rpy="-6.123E-17 0 0" xyz="${x_loc} ${y_loc + shaft_w/2 - 0.01} ${shaft_h/2 + dummy_r - agv_height/2 - hollow_h}" />
       <parent link="${parent}" />
       <child link="${name}_shaft_link" />

Commit message: change the base_link to its actual inertia

File: urdf/agv2.urdf.xacro (robot description, xacro)
@@ -22,7 +22,14 @@
   </joint>
   <link name="base_link">
+<!--
     <xacro:box_inertial mass="50" x="0.645" y="1.099" z="0.28">
       <origin rpy="0 0 ${M_PI/2}" xyz="0 0 0" />
     </xacro:box_inertial>
+-->
+    <inertial>
+      <origin rpy="0 0 ${M_PI/2}" xyz="0 0 0"/>
+      <mass value="50.0"/>
+      <inertia ixx="0.007081" ixy="-0.000118" ixz="-7.4538e-07" iyy="0.017373" iyz="0.000001" izz="0.022258"/>
+    </inertial>
     <visual>
       <origin xyz="0 0 0" rpy="0 0 ${M_PI/2}" />

Commit message: change the move limit axis for the ros joint

File: urdf/agv2.urdf.xacro (robot description, xacro)
@@ -47,13 +47,13 @@
   </link>
   <!-- rod -->
+  <property name="rod_r" value="0.0136" />
+  <property name="rod_h" value="0.060" />
   <joint name="rod_joint" type="prismatic">
-    <axis xyz="0 1 0"/>
-    <limit effort="1000.0" velocity="0.5"/>
+    <axis xyz="0 0 1"/>
+    <limit effort="1000.0" velocity="0.5" lower="0" upper="${rod_h}"/>
     <origin xyz="0 0.42475 ${agv_height/2 - rod_h/2}" rpy="0 0 0" />
     <parent link="base_link"/>
     <child link="rod_link" />
   </joint>
-  <property name="rod_r" value="0.0136" />
-  <property name="rod_h" value="0.060" />
   <link name="rod_link">
         <xacro:cylinder_inertial mass="0.1" radius="${rod_r}" length="${rod_h}">

Commit message: add transmission for the lift rod

File: urdf/agv2.urdf.xacro (robot description, xacro)
@@ -91,21 +91,14 @@
   <xacro:dummy_wheel name="rr_wheel" parent="base_link" x_loc="${BASE_DUMMY_R*-1}" y_loc="-0.42475">
   </xacro:dummy_wheel>
-<!--
-  <joint name="screen_joint" type="fixed"> ${drive_wheel_r - agv_height/2 - hollow_h} ${shaft_h + dummy_r - agv_height/2 - hollow_h}
-    <axis xyz="0 0 1"/>
-    <limit effort="1000.0" lower="-3.1415" upper="3.1415" velocity="0.5"/>
-    <origin xyz="0 -0.01 0.3" rpy="${0.1745*6} 0 0"/>
-    <parent link="chest_link"/>
-    <child link="screen_link"/>
-  </joint>
-  <link name="screen_link">
-    <visual>
-      <origin xyz="0 -0.055 0" rpy="0 0 0" />
-      <geometry>
-        <cylinder length="0.01" radius="0.09"/>
-      </geometry>
-      <material name="Orange"/>
-    </visual>
-  </link>
--->
+  <!-- Transmission -->
+  <transmission name="rod_tran">
+    <type>transmission_interface/SimpleTransmission</type>
+    <joint name="rod_joint">
+      <hardwareInterface>EffortJointInterface</hardwareInterface>
+    </joint>
+    <actuator name="rod_linear_motor">
+      <hardwareInterface>EffortJointInterface</hardwareInterface>
+      <mechanicalReduction>1</mechanicalReduction>
+    </actuator>
+  </transmission>
 </robot>

Commit message: make model heavier
more stable

File: urdf/agv2.urdf.xacro (robot description, xacro)
@@ -29,5 +29,5 @@
     <inertial>
       <origin rpy="0 0 ${M_PI/2}" xyz="0 0 0"/>
-      <mass value="50.0"/>
+      <mass value="100.0"/>
       <inertia ixx="0.007081" ixy="-0.000118" ixz="-7.4538e-07" iyy="0.017373" iyz="0.000001" izz="0.022258"/>
     </inertial>
@@ -57,5 +57,5 @@
   </joint>
   <link name="rod_front_link">
-        <xacro:cylinder_inertial mass="0.1" radius="${rod_r}" length="${rod_h}">
+        <xacro:cylinder_inertial mass="1.0" radius="${rod_r}" length="${rod_h}">
           <origin rpy="0 0 0" xyz="0 0 0" />
         </xacro:cylinder_inertial>
@@ -82,5 +82,5 @@
   </joint>
   <link name="rod_rear_link">
-        <xacro:cylinder_inertial mass="0.1" radius="${rod_r}" length="${rod_h}">
+        <xacro:cylinder_inertial mass="1.0" radius="${rod_r}" length="${rod_h}">
           <origin rpy="0 0 0" xyz="0 0 0" />
         </xacro:cylinder_inertial>
