Commit message: minor modify the imu description

File: urdf/imu.gazebo.xacro (robot description, xacro)
@@ -14,5 +14,4 @@
       <bodyName>imu_link</bodyName>
       <topicName>imu_data</topicName>
-      <frameId>imu</frameId>
     </plugin>
   </gazebo>

File: urdf/imu.urdf.xacro (robot description, xacro)
@@ -3,5 +3,5 @@
   <joint name="imu_joint" type="fixed">
     <axis xyz="0 1 0" />
-    <origin xyz="0 0 0" rpy="0 0 ${-M_PI/2}"/>
+    <origin xyz="0 0 0" rpy="0 0 0"/>
     <parent link="base_link"/>
     <child link="imu_link"/>
