Commit message: make the agv body looks transparant

File: urdf/agv2.gazebo.xacro (robot description, xacro)
@@ -52,5 +52,8 @@
     <mu1>10</mu1>
     <mu2>10</mu2>
+    <material>Gazebo/RedTransparent</material>
+<!--
     <material>Gazebo/WoodPallet</material>
+-->
   </gazebo>
   <gazebo reference="ground_plane">

Commit message: fixed the shelf unstable bug
and model sinking into ground plane problem

File: urdf/agv2.gazebo.xacro (robot description, xacro)
@@ -57,22 +57,3 @@
 -->
   </gazebo>
-  <gazebo reference="ground_plane">
-     <surface>
-        <friction>
-            <ode>
-                <mu>0.8</mu>
-            </ode>
-        </friction>
-        <bounce>
-            <restitution_coefficient>0.0</restitution_coefficient>
-        </bounce>
-        <contact>
-            <ode>
-                <kp>50000</kp>
-                <kd>5000</kd>
-                <max_vel>0</max_vel>
-            </ode>
-        </contact>
-    </surface>
-  </gazebo>
 </robot>

File: urdf/shelf.gazebo.xacro (robot description, xacro)
@@ -2,6 +2,6 @@
 <robot>
   <gazebo reference="base_link">
-    <kp>500000.0</kp>
-    <kd>10.0</kd>
+    <kp>1000000000</kp>
+    <kd>500000</kd>
     <mu1>10</mu1>
     <mu2>10</mu2>
@@ -11,22 +11,3 @@
 -->
   </gazebo>
-  <gazebo reference="ground_plane">
-     <surface>
-        <friction>
-            <ode>
-                <mu>0.8</mu>
-            </ode>
-        </friction>
-        <bounce>
-            <restitution_coefficient>0.0</restitution_coefficient>
-        </bounce>
-        <contact>
-            <ode>
-                <kp>50000</kp>
-                <kd>5000</kd>
-                <max_vel>0</max_vel>
-            </ode>
-        </contact>
-    </surface>
-  </gazebo>
 </robot>

File: urdf/shelf.urdf.xacro (robot description, xacro)
@@ -9,7 +9,5 @@
   <xacro:include filename="$(find agv2_description)/urdf/controller.gazebo" />
 -->
-<!--
   <xacro:include filename="$(find agv2_description)/urdf/wheel_shelf.urdf.xacro" />
--->
 <!--
   <xacro:include filename="$(find agv2_description)/urdf/laser.urdf.xacro" />
@@ -18,23 +16,30 @@
   <link name="base_footprint"/>
   <!-- Base -->
-  <property name="agv_height" value="0.268" />
-  <property name="hollow_h" value="0.34" />
+  <property name="agv_height" value="0.34" />
+  <property name="hollow_h" value="${0.1076}" />
   <joint name="base_joint" type="fixed">
     <axis xyz="0 0 1"/>
     <limit effort="1000.0" velocity="0.5"/>
-    <origin xyz="0 0 ${hollow_h}" rpy="0 0 0" />
+    <origin xyz="0 0 ${hollow_h + agv_height}" rpy="0 0 0" />
     <parent link="base_footprint"/>
     <child link="base_link" />
   </joint>
   <link name="base_link">
+<!--
     <inertial>
       <origin rpy="${M_PI/2} 0 0" xyz="0 0 0"/>
       <mass value="1.0"/>
-      <inertia ixx="0.0006699485" ixy="0.0" ixz="0.0" iyy="0.0010901" iyz="0.0" izz="0.0004378"/>
+      <inertia ixx="0.051828" ixy="0.0" ixz="0.0" iyy="0.088812" iyz="0.00012" izz="0.04517"/>
+    </inertial>
+-->
+    <inertial>
+      <origin rpy="${M_PI/2} 0 0" xyz="0 0 0"/>
+      <mass value="200.0"/>
+      <inertia ixx="0.0052406" ixy="0.0" ixz="0.0" iyy="0.0095404" iyz="0.00000025838" izz="0.004385"/>
     </inertial>
     <visual>
       <origin xyz="0 0 0" rpy="${M_PI/2} 0 0" />
         <geometry>
-          <mesh filename="package://agv2_description/meshes/pallet_spring_supp_brk_100kg.stl" scale="0.001 0.001 0.001"/>
+          <mesh filename="package://agv2_description/meshes/pallet_spring_supp_brk_100kg_with_top.stl" scale="0.001 0.001 0.001"/>
         </geometry>
     </visual>
@@ -42,20 +47,19 @@
       <origin xyz="0 0 0" rpy="${M_PI/2} 0 0" />
         <geometry>
-          <mesh filename="package://agv2_description/meshes/pallet_spring_supp_brk_100kg.stl" scale="0.001 0.001 0.001"/>
+          <mesh filename="package://agv2_description/meshes/pallet_spring_supp_brk_100kg_with_top.stl" scale="0.001 0.001 0.001"/>
         </geometry>
     </collision>
   </link>
   <!-- wheel -->
-  <property name="BASE_DUMMY_R" value="0.553"/>
-<!--
-  <xacro:dummy_wheel name="lf_wheel" parent="base_link" x_loc="${BASE_DUMMY_R}" y_loc="0.592">
+  <property name="BASE_DUMMY_R" value="${0.553 + 0.0115}"/>
+  <property name="BASE_DUMMY_L" value="${0.592 + 0.0115}"/>
+  <xacro:dummy_wheel name="lf_wheel" parent="base_link" x_loc="${BASE_DUMMY_R}" x_dir="1" y_loc="${BASE_DUMMY_L}" y_dir="1">
   </xacro:dummy_wheel>
-  <xacro:dummy_wheel name="rf_wheel" parent="base_link" x_loc="${BASE_DUMMY_R*-1}" y_loc="0.592">
+  <xacro:dummy_wheel name="rf_wheel" parent="base_link" x_loc="${BASE_DUMMY_R}" x_dir="-1" y_loc="${BASE_DUMMY_L}" y_dir="1">
   </xacro:dummy_wheel>
-  <xacro:dummy_wheel name="lr_wheel" parent="base_link" x_loc="${BASE_DUMMY_R}" y_loc="-0.592">
+  <xacro:dummy_wheel name="lr_wheel" parent="base_link" x_loc="${BASE_DUMMY_R}" x_dir="1" y_loc="${BASE_DUMMY_L}" y_dir="-1">
   </xacro:dummy_wheel>
-  <xacro:dummy_wheel name="rr_wheel" parent="base_link" x_loc="${BASE_DUMMY_R*-1}" y_loc="-0.592">
+  <xacro:dummy_wheel name="rr_wheel" parent="base_link" x_loc="${BASE_DUMMY_R}" x_dir="-1" y_loc="${BASE_DUMMY_L}" y_dir="-1">
   </xacro:dummy_wheel>
--->
 <!--
   <joint name="screen_joint" type="fixed"> ${drive_wheel_r - agv_height/2 - hollow_h} ${shaft_h + dummy_r - agv_height/2 - hollow_h}

File: urdf/wheel_shelf.urdf.xacro (robot description, xacro)
@@ -32,8 +32,8 @@
   <property name="dummy_w" value="0.033" />
   <property name="shaft_h" value="0.0695" />
-  <property name="shaft_w" value="0.033" />
-  <xacro:macro name="dummy_wheel" params="name parent x_loc y_loc">
+  <property name="shaft_w" value="${0.033 + 0.02}" />
+  <xacro:macro name="dummy_wheel" params="name parent x_loc x_dir y_loc y_dir">
     <link name="${name}_shaft_link">
-        <xacro:box_inertial mass="0.1" x="${shaft_w}" y="${dummy_w}" z="${shaft_h}">
+        <xacro:box_inertial mass="4.0" x="${shaft_w}" y="${shaft_w}" z="${shaft_h}">
           <origin rpy="0 0 0" xyz="0 0 0" />
         </xacro:box_inertial>
@@ -41,5 +41,5 @@
         <origin rpy="0 0 0" xyz="0 0 0" />
         <geometry>
-          <box size="${shaft_w} ${dummy_w} ${shaft_h}"/>
+          <box size="${shaft_w} ${shaft_w} ${shaft_h}"/>
         </geometry>
         <material name="">
@@ -50,5 +50,5 @@
         <origin rpy="0 0 0" xyz="0 0 0" />
         <geometry>
-          <box size="${shaft_w} ${dummy_w} ${shaft_h}"/>
+          <box size="${shaft_w} ${shaft_w} ${shaft_h}"/>
         </geometry>
         <material name="">
@@ -58,5 +58,5 @@
     </link>
     <link name="${name}_dummy_wheel">
-        <xacro:cylinder_inertial mass="0.1" radius="${dummy_r}" length="${dummy_w}">
+        <xacro:cylinder_inertial mass="4.0" radius="${dummy_r}" length="${dummy_w}">
           <origin rpy="0 ${M_PI/2} 0" xyz="0 0 0" />
         </xacro:cylinder_inertial>
@@ -78,8 +78,9 @@
     </link>
     <joint name="${name}_joint_shaft" type="continuous">
-      <origin rpy="-6.123E-17 0 0" xyz="${x_loc} ${y_loc + shaft_w/2 - 0.01} 0" />
+      <origin rpy="-6.123E-17 0 0" xyz="${(x_loc - shaft_w/2)*x_dir} ${(y_loc - shaft_w/2)*y_dir} ${(agv_height + 0.01)*-1}" />
       <parent link="${parent}" />
       <child link="${name}_shaft_link" />
       <axis xyz="0 0 1" />
+      <dynamics damping="0.9" friction="0.9" />
     </joint>
     <joint name="${name}_joint_roller" type="continuous">
@@ -90,16 +91,18 @@
     </joint>
     <gazebo reference="${name}_dummy_wheel">
-      <kp>500000.0</kp>
-      <kd>10.0</kd>
-      <mu1>0.01</mu1>
-      <mu2>0.01</mu2>
+      <kp>1000000000.0</kp>
+      <kd>500000.0</kd>
+      <mu1>1000.0</mu1>
+      <mu2>500.0</mu2>
+      <fdir1>1 0 0</fdir1>
     </gazebo>
     <gazebo reference="${name}_shaft_link">
-      <mu1>50</mu1>
-      <mu2>10</mu2>
-<!--
-      <dampingFactor>0.1</dampingFactor> ${shaft_h/2 + dummy_r - agv_height/2 - hollow_h}
--->
+      <kp>1000000000.0</kp>
+      <kd>500000.0</kd>
+      <mu1>1.0</mu1>
+      <mu2>1.0</mu2>
       <fdir1>0 0 1</fdir1>
+      <material>Gazebo/RedTransparent</material>
+      <dampingFactor>0.2</dampingFactor>
     </gazebo>
   </xacro:macro>

Commit message: add a rod in agv2
The rod is used to connect to the shelf

File: urdf/agv2.gazebo.xacro (robot description, xacro)
@@ -57,3 +57,12 @@
 -->
   </gazebo>
+  <gazebo reference="rod_link">
+    <kp>500000.0</kp>
+    <kd>10.0</kd>
+    <mu1>0.1</mu1>
+    <mu2>0.1</mu2>
+    <maxVel>1.0</maxVel>
+    <minDepth>0.003</minDepth>
+    <material>Gazebo/WoodPallet</material>
+  </gazebo>
 </robot>

File: urdf/agv2.urdf.xacro (robot description, xacro)
@@ -46,4 +46,31 @@
     </collision>
   </link>
+  <!-- rod -->
+  <joint name="rod_joint" type="prismatic">
+    <axis xyz="0 1 0"/>
+    <limit effort="1000.0" velocity="0.5"/>
+    <origin xyz="0 0.42475 ${agv_height/2 - rod_h/2}" rpy="0 0 0" />
+    <parent link="base_link"/>
+    <child link="rod_link" />
+  </joint>
+  <property name="rod_r" value="0.0136" />
+  <property name="rod_h" value="0.060" />
+  <link name="rod_link">
+        <xacro:cylinder_inertial mass="0.1" radius="${rod_r}" length="${rod_h}">
+          <origin rpy="0 0 0" xyz="0 0 0" />
+        </xacro:cylinder_inertial>
+    <visual>
+      <origin xyz="0 0 0" rpy="0 0 0" />
+        <geometry>
+          <cylinder length="${rod_h}" radius="${rod_r}"/>
+        </geometry>
+    </visual>
+    <collision>
+      <origin xyz="0 0 0" rpy="0 0 0" />
+        <geometry>
+          <cylinder length="${rod_h}" radius="${rod_r}"/>
+        </geometry>
+    </collision>
+  </link>
   <!-- wheel -->
   <property name="BASE_R" value="0.251"/>

Commit message: add two rods and put them on correct position

File: urdf/agv2.gazebo.xacro (robot description, xacro)
@@ -57,5 +57,14 @@
 -->
   </gazebo>
-  <gazebo reference="rod_link">
+  <gazebo reference="rod_front_link">
+    <kp>500000.0</kp>
+    <kd>10.0</kd>
+    <mu1>0.1</mu1>
+    <mu2>0.1</mu2>
+    <maxVel>1.0</maxVel>
+    <minDepth>0.003</minDepth>
+    <material>Gazebo/WoodPallet</material>
+  </gazebo>
+  <gazebo reference="rod_rare_link">
     <kp>500000.0</kp>
     <kd>10.0</kd>

File: urdf/agv2.urdf.xacro (robot description, xacro)
@@ -46,15 +46,40 @@
     </collision>
   </link>
-  <!-- rod -->
+  <!-- rod front -->
   <property name="rod_r" value="0.0136" />
   <property name="rod_h" value="0.060" />
-  <joint name="rod_joint" type="prismatic">
+  <joint name="rod_front_joint" type="prismatic">
     <axis xyz="0 0 1"/>
     <limit effort="1000.0" velocity="0.5" lower="0" upper="${rod_h}"/>
-    <origin xyz="0 0.42475 ${agv_height/2 - rod_h/2}" rpy="0 0 0" />
+    <origin xyz="0 -0.398 ${agv_height/2 - rod_h/2}" rpy="0 0 0" />
     <parent link="base_link"/>
-    <child link="rod_link" />
+    <child link="rod_front_link" />
   </joint>
-  <link name="rod_link">
+  <link name="rod_front_link">
+        <xacro:cylinder_inertial mass="0.1" radius="${rod_r}" length="${rod_h}">
+          <origin rpy="0 0 0" xyz="0 0 0" />
+        </xacro:cylinder_inertial>
+    <visual>
+      <origin xyz="0 0 0" rpy="0 0 0" />
+        <geometry>
+          <cylinder length="${rod_h}" radius="${rod_r}"/>
+        </geometry>
+    </visual>
+    <collision>
+      <origin xyz="0 0 0" rpy="0 0 0" />
+        <geometry>
+          <cylinder length="${rod_h}" radius="${rod_r}"/>
+        </geometry>
+    </collision>
+  </link>
+  <!-- rod rares -->
+  <joint name="rod_rare_joint" type="prismatic">
+    <axis xyz="0 0 1"/>
+    <limit effort="1000.0" velocity="0.5" lower="0" upper="${rod_h}"/>
+    <origin xyz="0 0.340 ${agv_height/2 - rod_h/2}" rpy="0 0 0" />
+    <parent link="base_link"/>
+    <child link="rod_rare_link" />
+  </joint>
+  <link name="rod_rare_link">
         <xacro:cylinder_inertial mass="0.1" radius="${rod_r}" length="${rod_h}">
           <origin rpy="0 0 0" xyz="0 0 0" />
@@ -92,10 +117,20 @@
   </xacro:dummy_wheel>
   <!-- Transmission -->
-  <transmission name="rod_tran">
+  <transmission name="rod_front_tran">
     <type>transmission_interface/SimpleTransmission</type>
-    <joint name="rod_joint">
+    <joint name="rod_front_joint">
       <hardwareInterface>EffortJointInterface</hardwareInterface>
     </joint>
-    <actuator name="rod_linear_motor">
+    <actuator name="rod_front_linear_motor">
+      <hardwareInterface>EffortJointInterface</hardwareInterface>
+      <mechanicalReduction>1</mechanicalReduction>
+    </actuator>
+  </transmission>
+  <transmission name="rod_rare_tran">
+    <type>transmission_interface/SimpleTransmission</type>
+    <joint name="rod_rare_joint">
+      <hardwareInterface>EffortJointInterface</hardwareInterface>
+    </joint>
+    <actuator name="rod_rare_linear_motor">
       <hardwareInterface>EffortJointInterface</hardwareInterface>
       <mechanicalReduction>1</mechanicalReduction>

Commit message: fixed typo

File: urdf/agv2.gazebo.xacro (robot description, xacro)
@@ -66,5 +66,5 @@
     <material>Gazebo/WoodPallet</material>
   </gazebo>
-  <gazebo reference="rod_rare_link">
+  <gazebo reference="rod_rear_link">
     <kp>500000.0</kp>
     <kd>10.0</kd>

File: urdf/agv2.urdf.xacro (robot description, xacro)
@@ -73,13 +73,13 @@
     </collision>
   </link>
-  <!-- rod rares -->
-  <joint name="rod_rare_joint" type="prismatic">
+  <!-- rod rears -->
+  <joint name="rod_rear_joint" type="prismatic">
     <axis xyz="0 0 1"/>
     <limit effort="1000.0" velocity="0.5" lower="0" upper="${rod_h}"/>
     <origin xyz="0 0.340 ${agv_height/2 - rod_h/2}" rpy="0 0 0" />
     <parent link="base_link"/>
-    <child link="rod_rare_link" />
+    <child link="rod_rear_link" />
   </joint>
-  <link name="rod_rare_link">
+  <link name="rod_rear_link">
         <xacro:cylinder_inertial mass="0.1" radius="${rod_r}" length="${rod_h}">
           <origin rpy="0 0 0" xyz="0 0 0" />
@@ -127,10 +127,10 @@
     </actuator>
   </transmission>
-  <transmission name="rod_rare_tran">
+  <transmission name="rod_rear_tran">
     <type>transmission_interface/SimpleTransmission</type>
-    <joint name="rod_rare_joint">
+    <joint name="rod_rear_joint">
       <hardwareInterface>EffortJointInterface</hardwareInterface>
     </joint>
-    <actuator name="rod_rare_linear_motor">
+    <actuator name="rod_rear_linear_motor">
       <hardwareInterface>EffortJointInterface</hardwareInterface>
       <mechanicalReduction>1</mechanicalReduction>

Commit message: trun agv2 back from the yaw not consistency

File: urdf/agv2.gazebo.xacro (robot description, xacro)
@@ -6,5 +6,5 @@
     <mu1>100</mu1>
     <mu2>10</mu2>
-    <fdir1>1 0 0</fdir1>
+    <fdir1>0 1 0</fdir1>
     <maxVel>1.0</maxVel>
     <minDepth>0.003</minDepth>
@@ -16,5 +16,5 @@
     <mu1>100</mu1>
     <mu2>10</mu2>
-    <fdir1>1 0 0</fdir1>
+    <fdir1>0 1 0</fdir1>
     <maxVel>1.0</maxVel>
     <minDepth>0.003</minDepth>

File: urdf/agv2.urdf.xacro (robot description, xacro)
@@ -35,5 +35,5 @@
     </inertial>
     <visual>
-      <origin xyz="0 0 0" rpy="0 0 ${M_PI/2}" />
+      <origin xyz="0 0 0" rpy="0 0 0" />
         <geometry>
           <mesh filename="package://agv2_description/meshes/agv_black.dae" />
@@ -42,5 +42,5 @@
     </visual>
     <collision>
-      <origin xyz="0 0 0" rpy="0 0 ${M_PI/2}" />
+      <origin xyz="0 0 0" rpy="0 0 0" />
         <geometry>
           <mesh filename="package://agv2_description/meshes/agv_black.stl" />
@@ -54,5 +54,5 @@
     <axis xyz="0 0 1"/>
     <limit effort="1000.0" velocity="0.5" lower="0" upper="${rod_h}"/>
-    <origin xyz="0 -0.398 ${agv_height/2 - rod_h/2}" rpy="0 0 0" />
+    <origin xyz="0.340 0 ${agv_height/2 - rod_h/2}" rpy="0 0 0" />
     <parent link="base_link"/>
     <child link="rod_front_link" />
@@ -79,5 +79,5 @@
     <axis xyz="0 0 1"/>
     <limit effort="1000.0" velocity="0.5" lower="0" upper="${rod_h}"/>
-    <origin xyz="0 0.340 ${agv_height/2 - rod_h/2}" rpy="0 0 0" />
+    <origin xyz="-0.398 0 ${agv_height/2 - rod_h/2}" rpy="0 0 0" />
     <parent link="base_link"/>
     <child link="rod_rear_link" />
@@ -105,16 +105,16 @@
   <property name="drive_wheel_r" value="0.08" />
   <xacro:wheel name="l_wheel" parent="base_link" radius="${drive_wheel_r}" width="0.05">
-    <origin rpy="-6.123E-17 0 0" xyz="${BASE_R} 0.0 ${drive_wheel_r - agv_height/2 - hollow_h}" />
+    <origin rpy="-6.123E-17 0 0" xyz=" 0.0 ${BASE_R} ${drive_wheel_r - agv_height/2 - hollow_h}" />
   </xacro:wheel>
   <xacro:wheel name="r_wheel" parent="base_link" radius="${drive_wheel_r}" width="0.05">
-    <origin rpy="-6.123E-17 0 0" xyz="${BASE_R*-1} 0.0 ${drive_wheel_r - agv_height/2 - hollow_h}" />
+    <origin rpy="-6.123E-17 0 0" xyz=" 0.0 ${BASE_R*-1} ${drive_wheel_r - agv_height/2 - hollow_h}" />
   </xacro:wheel>
-  <xacro:dummy_wheel name="lf_wheel" parent="base_link" x_loc="${BASE_DUMMY_R}" y_loc="0.4275">
+  <xacro:dummy_wheel name="lf_wheel" parent="base_link" y_loc="${BASE_DUMMY_R}" x_loc="0.4275">
   </xacro:dummy_wheel>
-  <xacro:dummy_wheel name="rf_wheel" parent="base_link" x_loc="${BASE_DUMMY_R*-1}" y_loc="0.4275">
+  <xacro:dummy_wheel name="rf_wheel" parent="base_link" y_loc="${BASE_DUMMY_R*-1}" x_loc="0.4275">
   </xacro:dummy_wheel>
-  <xacro:dummy_wheel name="lr_wheel" parent="base_link" x_loc="${BASE_DUMMY_R}" y_loc="-0.42475">
+  <xacro:dummy_wheel name="lr_wheel" parent="base_link" y_loc="${BASE_DUMMY_R}" x_loc="-0.42475">
   </xacro:dummy_wheel>
-  <xacro:dummy_wheel name="rr_wheel" parent="base_link" x_loc="${BASE_DUMMY_R*-1}" y_loc="-0.42475">
+  <xacro:dummy_wheel name="rr_wheel" parent="base_link" y_loc="${BASE_DUMMY_R*-1}" x_loc="-0.42475">
   </xacro:dummy_wheel>
   <!-- Transmission -->

File: urdf/laser.urdf.xacro (robot description, xacro)
@@ -6,5 +6,5 @@
     may not be the reall pose, it is just an estimation
 -->
-    <origin xyz="0 -0.50 0.14" rpy="0 0 ${-M_PI/2}"/>
+    <origin xyz="0.50 0 0.14" rpy="0 0 0"/>
     <parent link="base_link"/>
     <child link="laser_link"/>

File: urdf/wheel_agv.urdf.xacro (robot description, xacro)
@@ -4,8 +4,8 @@
     <link name="${name}_link">
         <xacro:cylinder_inertial mass="0.1" radius="${radius}" length="${width}">
-          <origin rpy="0 ${M_PI/2} 0" xyz="0 0 0" />
+          <origin rpy="${M_PI/2} 0 0" xyz="0 0 0" />
         </xacro:cylinder_inertial>
       <visual>
-        <origin rpy="0 ${M_PI/2} 0" xyz="0 0 0" />
+        <origin rpy="${M_PI/2} 0 0" xyz="0 0 0" />
         <geometry>
           <cylinder length="${width}" radius="${radius}"/>
@@ -16,5 +16,5 @@
       </visual>
       <collision>
-        <origin rpy="0 ${M_PI/2} 0" xyz="0 0 0" />
+        <origin rpy="${M_PI/2} 0 0" xyz="0 0 0" />
         <geometry>
           <cylinder length="${width}" radius="${radius}"/>
@@ -26,5 +26,5 @@
       <parent link="${parent}" />
       <child link="${name}_link" />
-      <axis xyz="1 0 0" />
+      <axis xyz="0 1 0" />
     <limit effort="108.85" velocity="34.8" /></joint>
   </xacro:macro>
